Commit message: Aggiunti modelli guardia e thief

File: description/urdf/thief.xacro (robot description, xacro)
@@ -1,4 +1,4 @@
 <?xml version="1.0"?>
-<robot name="nostop" xmlns:xacro="http://www.ros.org/wiki/xacro">
+<robot name="nostop_thief" xmlns:xacro="http://www.ros.org/wiki/xacro">
         <!-- Put here the robot description -->
 <xacro:property name="PI" value="3.1415926535897931"/>
@@ -36,5 +36,5 @@
       <box size="${chassisLength} ${chassisWidth} ${chassisHeight}"/>
     </geometry>
-    <material name="orange"/>
+    <material name="blue"/>
   </visual>
   <inertial>
@@ -45,5 +45,5 @@
 </link>
 <gazebo reference="chassis">
-  <material>Gazebo/Orange</material>
+  <material>Gazebo/Blue</material>
 </gazebo>
 <joint name="fixed" type="fixed">
